File: eagle/projects/ray/ray.brd (EAGLE design)
At the start: 17.8 x 425.4 mm, 4 parts

Commit message: make solder pads for LED strips more forgiving
Parts:
- added L1, R1: 1X4SMT, adafruit:1X4-SMT
Connections:
- net 5V: now also L1.1, R1.1
- net GND: now also L1.4, R1.4
- net RC: now also R1.2
- net RD: now also R1.3
- net TTC: now also L1.2
- net TTD: now also L1.3
Routing:
- net 5V: track 50.0 -> 60.1 mm, vias 18 -> 19
- net GND: track 42.9 -> 50.6 mm, vias 18 -> 19
- net TTD: track 436.2 -> 440.7 mm, vias 6 -> 10
- net RC: track 27.6 -> 32.0 mm, vias 0 -> 4
- net TTC: track 429.7 -> 433.5 mm
- net RD: track 8.76 -> 12.6 mm
- added copper zone on layer 1, net RC
- added copper zone on layer 1, net RD
