File: eagle/projects/ray/ray0.brd (EAGLE design)
At the start: 17.8 x 445.5 mm, 8 parts, among them CN1 1X4SMT, CN2 1X4SMT

Commit message: make solder pads for LED strips more forgiving
Parts:
- added L1, R1: 1X4SMT, adafruit:1X4-SMT
- JP1: value (none) -> input
Connections:
- net 5V: now also L1.1, R1.1
- net GND: now also L1.4, R1.4
- net LC: now also L1.2
- net LD: now also L1.3
- net RC: now also R1.2
- net RD: now also R1.3
Routing:
- net GND: track 10.9 -> 31.8 mm, vias 40 -> 36
- net 5V: track 39.0 -> 31.4 mm, vias 22 -> 25
- net RC: track 28.8 -> 32.9 mm, vias 0 -> 4
- net LD: track 0.00 -> 3.81 mm
- net LC: track 0.00 -> 3.81 mm
- net RD: track 8.76 -> 12.6 mm
- net TRC: track 226.9 -> 229.5 mm, vias 0 -> 4
- net TRD: track 231.8 -> 234.4 mm, vias 0 -> 4
- added copper zone on layer 1, net RC
- added copper zone on layer 1, net RD
